File: eCAD/lick-detector/schmitt-trigger.kicad_sch (KiCad schematic)
At the start: 8 parts, among them J9 J_PinHeader_01x02_2.54_V, U2 OPA2365

Commit message: Number of upgrades complete: - Lower amplitude sine wave generator - Improved debug connector layout - Brightness of LED decreased - README updated with guide and areas for documentation - .gitignore added to ignore backup files and temporary files
Parts:
- renumbered RV3 to RV2
Changed lines of the file:
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@@
 		(in_pos_files yes)
 		(dnp no)
-		(property "Reference" "RV3"
+		(property "Reference" "RV2"
 			(at 153.67 101.6 90)
 			(show_name no)
@@
 			(project "lick-detector"
 				(path "/815e9fa1-5cc8-45e1-9d34-77c5548ab2a8/377e8981-2ca9-41bf-baa8-910decf7c125"
-					(reference "RV3")
+					(reference "RV2")
 					(unit 1)
 				)
